Commit message: scoped include dir

File: urdf/terrain/terrain.xacro (robot description, xacro)
@@ -17,10 +17,10 @@
     <visual>
     <geometry>
-        <mesh filename="file://$(find ecn_auv_lab)/urdf/terrain/MangaliaTerrain.dae"  scale="1.0 1.0 5.0"/>
+        <mesh filename="package://ecn_auv_lab/urdf/terrain/MangaliaTerrain.dae"  scale="1.0 1.0 5.0"/>
       </geometry>
     </visual>
       <collision>
     <geometry>
-        <mesh filename="file://$(find ecn_auv_lab)/urdf/terrain/MangaliaTerrain.dae"  scale="1.0 1.0 5.0"/>
+        <mesh filename="package://ecn_auv_lab/urdf/terrain/MangaliaTerrain.dae"  scale="1.0 1.0 5.0"/>
       </geometry>
     </collision>
